File: kitchen-timer-phase-b-pcb-prototype/Phase_B_PCB_Prototype.kicad_pcb (KiCad board)
At the start: 2 copper layers, 83.9 x 58.5 mm, 49 parts, among them J1 USB_B_Mini, J2 AVR-ISP-6, J3 ESP Connector, U1 CA56-12EWA, U2 74HC595, U3 ATmega32U4-A, U4 USBLC6-2SC6, U5 LP2985-3.3, Y1 Crystal_GND24

Commit message: Enclosure and PCB updates
Parts:
- added REF**: MountingHole_3.2mm, Arduino_MountingHole:MountingHole_3.2mm, F.Cu at (130.8, 117.0)
- added REF**: MountingHole_3.2mm, Arduino_MountingHole:MountingHole_3.2mm, F.Cu at (73.5, 61.3)
- added REF**: MountingHole_3.2mm, Arduino_MountingHole:MountingHole_3.2mm, F.Cu at (89.4, 117.0)
- added REF**: MountingHole_3.2mm, Arduino_MountingHole:MountingHole_3.2mm, F.Cu at (151.8, 61.6)
- moved C9 13.9 mm to (142.5, 99.8), turned to 0 degrees
- moved C14 0.89 mm to (82.2, 111.1)
- moved U5 0.89 mm to (85.3, 111.1)
- moved C12 0.89 mm to (88.3, 111.3)
- moved C13 0.89 mm to (85.8, 108.6)
- moved J3 0.89 mm to (76.9, 106.6)
- moved R17 0.89 mm to (79.4, 110.7)
- moved S3 0.65 mm to (100.6, 110.4)
- moved R13 0.65 mm to (95.8, 111.4)
Routing:
- net Dig2: track 57.7 -> 49.8 mm
- net +5V: track 165.3 -> 162.6 mm
- net RST: track 92.2 -> 93.5 mm
- net TX: track 69.2 -> 70.1 mm
- net RX: track 68.0 -> 68.9 mm
- net GND: track 68.6 -> 67.7 mm, vias 31 -> 30
Other:
- board size 83.9 x 58.5 mm -> 83.9 x 61.3 mm

Commit message: Finished PCB and created gerber files
Parts:
- removed the REF** at (130.8, 117.0)
- removed the REF** at (73.5, 61.3)
- removed the REF** at (89.4, 117.0)
- removed the REF** at (151.8, 61.6)
- added REF**: MountingHole_3.2mm, Arduino_MountingHole:MountingHole_3.2mm, F.Cu at (151.9, 61.5)
- added REF**: MountingHole_3.2mm, Arduino_MountingHole:MountingHole_3.2mm, F.Cu at (92.8, 117.3)
- added REF**: MountingHole_3.2mm, Arduino_MountingHole:MountingHole_3.2mm, F.Cu at (73.7, 61.3)
- added REF**: MountingHole_3.2mm, Arduino_MountingHole:MountingHole_3.2mm, F.Cu at (128.3, 117.1)
Other:
- board text added: "+3.3V"
- board text added: "+5V"
- board text added: "------"
- board text added: "4x M3"
- board text added: "Alarm 0 1"
- board text added: "Dig 1"
- board text added: "Dig 4"
- board text added: "Embedded Systems"
- board text added: "GND"
- board text added: "Green Red"
- board text added: "Kitchen Timer"
- board text added: "Kitchen Timer v1.0 4/20/2023"
- board text added: "MISO"
- board text added: "MOSI"
- board text added: "Paused 1 1"
- board text added: "RST"
- board text added: "RX"
- board text added: "Running 1 0"
- board text added: "SCK"
- board text added: "TX"
- board text added: "Zach Bayler"
