File: kitchen-timer-phase-b-pcb-prototype/Phase_B_PCB_Prototype.kicad_sch (KiCad schematic)
At the start: 49 parts, among them J1 USB_B_Mini, J2 AVR-ISP-6, J3 ESP Connector, U1 CA56-12EWA, U2 74HC595, U3 ATmega32U4-A, U4 USBLC6-2SC6, U5 LP2985-3.3, Y1 Crystal_GND24

Commit message: Enclosure and PCB updates
Parts:
- C1: footprint Capacitor_SMD:C_0201_0603Metric -> Capacitor_SMD:C_0603_1608Metric
Changed lines of the file:
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@@
       (effects (font (size 1.27 1.27)) (justify left))
     )
-    (property "Footprint" "Capacitor_SMD:C_0201_0603Metric" (at 163.5252 109.22 0)
+    (property "Footprint" "Capacitor_SMD:C_0603_1608Metric" (at 163.5252 109.22 0)
       (effects (font (size 1.27 1.27)) hide)
     )

Commit message: Finished PCB and created gerber files
Changed lines of the file:
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@@
     (fill (type none))
+  )
+  (rectangle (start 186.69 187.96) (end 215.9 190.5)
+    (stroke (width -0.0001) (type default))
+    (fill (type color) (color 255 253 207 1))
   )
   (rectangle (start 246.38 128.27) (end 280.67 163.83)
